Commit message: Updating collision and ros2 control related things in ranger_mini_isaac.xacro

File: ranger/ranger_mini_v3/urdf/ranger_mini_isaac.xacro (robot description, xacro)
@@ -1,8 +1,24 @@
 <?xml version="1.0" encoding="utf-8"?>
 <robot name="ranger_mini_v3" xmlns:xacro="http://ros.org/wiki/xacro">
+  <!-- Chassis collision properties -->
+  <xacro:property name="chassis_x" value="0.74" />
+  <xacro:property name="chassis_y" value="0.5" />
+  <xacro:property name="chassis_z" value="0.1" />
+  <xacro:property name="chassis_z_origin" value="-0.04" />
+  <xacro:property name="chassis_sensor_x" value="0.02" />
+  <xacro:property name="chassis_sensor_y" value="0.25" />
+  <xacro:property name="chassis_sensor_z" value="0.1" />
+  <xacro:property name="chassis_sensor_x_origin" value="0.38" />
+  <xacro:property name="chassis_sensor_z_origin" value="-0.14" />
+  <!-- Wheel steering collision properties -->
+  <xacro:property name="wheel_steering_radius" value="0.035" />
+  <xacro:property name="wheel_steering_length" value="0.01" />
+  <!-- Wheel collision properties -->
+  <xacro:property name="wheel_radius" value="0.1" />
+  <xacro:property name="wheel_length" value="0.07" />
   <link name="base_link">
     <inertial>
+      <mass value="10" />
       <origin xyz="-0.0242698272228022 -0.0030308024613212 0.0544267444673498" rpy="0 0 0" />
-      <mass value="10" />
       <inertia ixx="0.1354" ixy="0.0" ixz="0.0" iyy="0.2417" iyz="0.0" izz="0.3085" />
     </inertial>
@@ -17,7 +33,14 @@
     </visual>
     <collision>
-      <origin xyz="0 0 0" rpy="3.141593 0 0" />
-      <geometry>
-        <mesh filename="package://ranger_mini_v3/meshes/ranger_mini3.dae" />
+      <origin xyz="0 0 ${chassis_z_origin}" rpy="0 0 0" />
+      <geometry>
+        <box size="${chassis_x} ${chassis_y} ${chassis_z}" />
+        <!-- <mesh filename="package://ranger_mini_v3/meshes/ranger_mini3.dae" /> -->
+      </geometry>
+    </collision>
+    <collision>
+      <origin xyz="${chassis_sensor_x_origin} 0 ${chassis_sensor_z_origin}" rpy="0 0 0" />
+      <geometry>
+        <box size="${chassis_sensor_x} ${chassis_sensor_y} ${chassis_sensor_z}" />
       </geometry>
     </collision>
@@ -25,6 +48,6 @@
   <link name="fr_steering_wheel_link">
     <inertial>
+      <mass value="1" />
       <origin xyz="1.8493E-05 1.2713E-06 0.043679" rpy="0 0 0" />
-      <mass value="1" />
       <inertia ixx="0.0063625" ixy="-1.0581E-07" ixz="-4.0831E-07" iyy="0.006363" iyz="-3.4944E-08" izz="0.010465" />
     </inertial>
@@ -39,7 +62,8 @@
     </visual>
     <collision>
-      <origin xyz="0 0 0" rpy="1.570796 0 0" />
-      <geometry>
-        <mesh filename="package://ranger_mini_v3/meshes/ranger_mini_v3_wheel_steering.dae" />
+      <origin xyz="0 0 0" rpy="0 0 0" />
+      <geometry>
+        <cylinder radius="${wheel_steering_radius}" length="${wheel_steering_length}" />
+        <!-- <mesh filename="package://ranger_mini_v3/meshes/ranger_mini_v3_wheel_steering.dae" /> -->
       </geometry>
     </collision>
@@ -50,5 +74,5 @@
     <child link="fr_steering_wheel_link" />
     <axis xyz="0 0 -1" />
-    <limit effort="5" velocity="6.28" lower="-2.1" upper="2.1" />
+    <limit effort="5" velocity="6.28" lower="-2.094" upper="2.094" />
   </joint>
   <link name="fr_wheel_link">
@@ -67,5 +91,7 @@
       <origin xyz="0 0 0" rpy="1.570796 0 0" />
       <geometry>
-        <mesh filename="package://ranger_mini_v3/meshes/ranger_mini_v3_wheel_tyre.dae" />
+        <cylinder radius="0.10" length="0.07" />
+        <cylinder radius="${wheel_radius}" length="${wheel_length}" />
+        <!-- <mesh filename="package://ranger_mini_v3/meshes/ranger_mini_v3_wheel_tyre.dae" /> -->
       </geometry>
       <contact>
@@ -84,6 +110,6 @@
   <link name="fl_steering_wheel_link">
     <inertial>
+      <mass value="1" />
       <origin xyz="-0.0017956 -9.6304E-08 0.043642" rpy="0 0 0" />
-      <mass value="1" />
       <inertia ixx="0.0063695" ixy="-2.1067E-08" ixz="-0.00016867" iyy="0.006363" iyz="-1.0301E-08" izz="0.010458" />
     </inertial>
@@ -98,7 +124,8 @@
     </visual>
     <collision>
-      <origin xyz="0 0 0" rpy="1.570796 0 3.141593" />
-      <geometry>
-        <mesh filename="package://ranger_mini_v3/meshes/ranger_mini_v3_wheel_steering.dae" />
+      <origin xyz="0 0 0" rpy="0 0 0" />
+      <geometry>
+        <cylinder radius="${wheel_steering_radius}" length="${wheel_steering_length}" />
+        <!-- <mesh filename="package://ranger_mini_v3/meshes/ranger_mini_v3_wheel_steering.dae" /> -->
       </geometry>
     </collision>
@@ -109,5 +136,5 @@
     <child link="fl_steering_wheel_link" />
     <axis xyz="0 0 -1" />
-    <limit effort="5" velocity="6.28" lower="-2.1" upper="2.1" />
+    <limit effort="5" velocity="6.28" lower="-2.094" upper="2.094" />
   </joint>
   <link name="fl_wheel_link">
@@ -126,5 +153,6 @@
       <origin xyz="0 0 0" rpy="-1.570796 0 0" />
       <geometry>
-        <mesh filename="package://ranger_mini_v3/meshes/ranger_mini_v3_wheel_tyre.dae" />
+        <cylinder radius="${wheel_radius}" length="${wheel_length}" />
+        <!-- <mesh filename="package://ranger_mini_v3/meshes/ranger_mini_v3_wheel_tyre.dae" /> -->
       </geometry>
       <contact>
@@ -143,6 +171,6 @@
   <link name="rl_steering_wheel_link">
     <inertial>
+      <mass value="1" />
       <origin xyz="-0.00017093 6.1255E-08 0.043678" rpy="0 0 0" />
-      <mass value="1" />
       <inertia ixx="0.0063627" ixy="-2.1069E-08" ixz="-1.587E-05" iyy="0.006363" iyz="9.3201E-09" izz="0.010465" />
     </inertial>
@@ -157,7 +185,8 @@
     </visual>
     <collision>
-      <origin xyz="0 0 0" rpy="1.570796 0.0 3.141593" />
-      <geometry>
-        <mesh filename="package://ranger_mini_v3/meshes/ranger_mini_v3_wheel_steering.dae" />
+      <origin xyz="0 0 0" rpy="0 0 0" />
+      <geometry>
+        <cylinder radius="${wheel_steering_radius}" length="${wheel_steering_length}" />
+        <!-- <mesh filename="package://ranger_mini_v3/meshes/ranger_mini_v3_wheel_steering.dae" /> -->
       </geometry>
     </collision>
@@ -168,5 +197,5 @@
     <child link="rl_steering_wheel_link" />
     <axis xyz="0 0 -1" />
-    <limit effort="5" velocity="6.28" lower="-2.1" upper="2.1" />
+    <limit effort="5" velocity="6.28" lower="-2.094" upper="2.094" />
   </joint>
   <link name="rl_wheel_link">
@@ -185,5 +214,6 @@
       <origin xyz="0 0 0" rpy="-1.570796 0 0" />
       <geometry>
-        <mesh filename="package://ranger_mini_v3/meshes/ranger_mini_v3_wheel_tyre.dae" />
+        <cylinder radius="${wheel_radius}" length="${wheel_length}" />
+        <!-- <mesh filename="package://ranger_mini_v3/meshes/ranger_mini_v3_wheel_tyre.dae" /> -->
       </geometry>
       <contact>
@@ -202,6 +232,6 @@
   <link name="rr_steering_wheel_link">
     <inertial>
+      <mass value="1" />
       <origin xyz="0.0 0.0 0.0" />
-      <mass value="1" />
       <inertia ixx="0.01" ixy="0.0" ixz="0.0" iyy="0.01" iyz="0.0" izz="0.01" />
     </inertial>
@@ -212,8 +242,7 @@
       </geometry>
     </visual>
-    <collision>
-      <origin xyz="0 0 0" rpy="1.570796 0 0" />
-      <geometry>
-        <mesh filename="package://ranger_mini_v3/meshes/ranger_mini_v3_wheel_steering.dae" />
+    <collision>01.570796 0 0" /> <geometry>
+        <cylinder radius="${wheel_steering_radius}" length="${wheel_steering_length}" />
+        <!-- <mesh filename="package://ranger_mini_v3/meshes/ranger_mini_v3_wheel_steering.dae" /> -->
       </geometry>
     </collision>
@@ -224,5 +253,5 @@
     <child link="rr_steering_wheel_link" />
     <axis xyz="0 0 -1" rpy="0 0 0" />
-    <limit effort="5" velocity="6.28" lower="-2.1" upper="2.1" />
+    <limit effort="5" velocity="6.28" lower="-2.094" upper="2.094" />
   </joint>
   <link name="rr_wheel_link">
@@ -241,5 +270,6 @@
       <origin xyz="0 0 0" rpy="1.570796 0 0" />
       <geometry>
-        <mesh filename="package://ranger_mini_v3/meshes/ranger_mini_v3_wheel_tyre.dae" />
+        <cylinder radius="${wheel_radius}" length="${wheel_length}" />
+        <!-- <mesh filename="package://ranger_mini_v3/meshes/ranger_mini_v3_wheel_tyre.dae" /> -->
       </geometry>
       <contact>
@@ -336,3 +366,61 @@
     </actuator>
   </transmission>
+  <!-- ros2_control Configuration -->
+  <ros2_control name="ranger_mini_control" type="system">
+    <hardware>
+      <plugin>topic_based_ros2_control/TopicBasedSystem</plugin>
+      <param name="joint_commands_topic">/robot_joint_command</param>
+      <param name="joint_states_topic">/robot_joint_states</param>
+      <param name="trigger_joint_command_threshold">0.001</param>
+      <param name="sum_wrapped_joint_states">true</param>
+    </hardware>
+    <joint name="fl_steering_joint">
+      <command_interface name="position" />
+      <command_interface name="velocity" />
+      <state_interface name="position" />
+      <state_interface name="velocity" />
+    </joint>
+    <joint name="fl_wheel">
+      <command_interface name="position" />
+      <command_interface name="velocity" />
+      <state_interface name="position" />
+      <state_interface name="velocity" />
+    </joint>
+    <joint name="fr_steering_joint">
+      <command_interface name="position" />
+      <command_interface name="velocity" />
+      <state_interface name="position" />
+      <state_interface name="velocity" />
+    </joint>
+    <joint name="fr_wheel">
+      <command_interface name="position" />
+      <command_interface name="velocity" />
+      <state_interface name="position" />
+      <state_interface name="velocity" />
+    </joint>
+    <joint name="rr_steering_joint">
+      <command_interface name="position" />
+      <command_interface name="velocity" />
+      <state_interface name="position" />
+      <state_interface name="velocity" />
+    </joint>
+    <joint name="rl_wheel">
+      <command_interface name="position" />
+      <command_interface name="velocity" />
+      <state_interface name="position" />
+      <state_interface name="velocity" />
+    </joint>
+    <joint name="rr_wheel">
+      <command_interface name="position" />
+      <command_interface name="velocity" />
+      <state_interface name="position" />
+      <state_interface name="velocity" />
+    </joint>
+    <joint name="rl_steering_joint">
+      <command_interface name="position" />
+      <command_interface name="velocity" />
+      <state_interface name="position" />
+      <state_interface name="velocity" />
+    </joint>
+  </ros2_control>
 </robot>
